File: hardware/RFBRD/file58A91AD0.sch (KiCad schematic (older format))
At the start: 26 parts

Commit message: Added bits of the RF Board, dumped to PCB.
Parts:
- added C23, C24: 3.183nF, Capacitors_SMD:C_0805, symbol C
- added J1: SMACONN, RFBRD:SMA_CONN, symbol SMACONN
- added L15: 16uH, Choke_SMD:Choke_SMD_12x12mm_h4.5mm, symbol INDUCTOR
- C10, C11, C12, C13, C14, C15, C16, C17, C18, C19, C20, C21, C22: renamed from C?; footprint (none) -> Capacitors_SMD:C_0805
- L10, L11, L12, L13, L14, L7, L8, L9: renamed from L?; footprint (none) -> Resistors_SMD:R_0805
- R1, R2, R3: renamed from R?; footprint (none) -> Resistors_SMD:R_0603
- RV1: renamed from RV?; value POT -> 47K; footprint (none) -> Air_Coils_SML_NEOSID:Neosid_Air-Coil_SML_2turn_HDM0231A
- U2: renamed from U?; footprint (none) -> RFBRD:SOT-89
Connections:
- net labels added: TX_OUT, TX_PASS
- net labels removed: 5W_OUT
- wire segments 49 -> 58
Other:
- moved on the sheet: C12, C14, L7, L9, R1, R2, RV1
