File: hardware/RFBRD/file58A91B00.sch (KiCad schematic (older format))
At the start: 0 parts

Commit message: Added bits of the RF Board, dumped to PCB.
Parts:
- added C30, C31: 3.183nF, Capacitors_SMD:C_0805, symbol C
- added C32, C33: 10nF, Capacitors_SMD:C_0805, symbol C
- added L19: 16uH, Choke_SMD:Choke_SMD_12x12mm_h4.5mm, symbol INDUCTOR
- added Q2: Q_NMOS_DGS, TO_SOT_Packages_SMD:SOT-23, symbol Q_NMOS_DGS
- added R10: 60.4, Resistors_SMD:R_0603, symbol R
- added R11: 50, Resistors_SMD:R_0603, symbol R
- added R12: 4, Resistors_SMD:R_0603, symbol R
- added R9: 309, Resistors_SMD:R_0603, symbol R
- added RV2: POT, RFBRD:J-FOOT_POT, symbol POT
Connections:
- new net: C31.1, C32.2, L19.2
- new net: C33.2, Q2.1 (D), R11.2
- new net: C32.1, Q2.2 (G), R10.1, R9.2
- new net: Q2.3 (S), R12.1
- new net: R11.1, R9.1, RV2.2
- new net 3V3: RV2.1
- new net GND: C30.2, C31.2, R10.2, R12.2, RV2.3
- new net RX_ANT: C30.1, L19.1
- new net RX_IN: C33.1
Changed lines of the file:
@@
 LIBS:contrib
 LIBS:valves
+LIBS:RFT
+LIBS:RFBRD-cache
 EELAYER 25 0
 EELAYER END
 $Descr A4 11693 8268
 encoding utf-8
-Sheet 1 6
+Sheet 5 6
 Title ""
 Date ""
@@
 Comment4 ""
 $EndDescr
+$Comp
+L C C30
+U 1 1 58C0D5DD
+P 2850 2450
+F 0 "C30" H 2875 2550 50  0000 L CNN
+F 1 "3.183nF" H 2875 2350 50  0000 L CNN
+F 2 "Capacitors_SMD:C_0805" H 2888 2300 50  0001 C CNN
+F 3 "" H 2850 2450 50  0000 C CNN
+	1    2850 2450
+	1    0    0    -1
+$EndComp
+$Comp
+L INDUCTOR L19
+U 1 1 58C0D616
+P 3250 2200
+F 0 "L19" V 3200 2200 50  0000 C CNN
+F 1 "16uH" V 3350 2200 50  0000 C CNN
+F 2 "Choke_SMD:Choke_SMD_12x12mm_h4.5mm" H 3250 2200 50  0001 C CNN
+F 3 "" H 3250 2200 50  0000 C CNN
+	1    3250 2200
+	0    -1   -1   0
+$EndComp
+$Comp
+L C C31
+U 1 1 58C0D651
+P 3650 2450
+F 0 "C31" H 3675 2550 50  0000 L CNN
+F 1 "3.183nF" H 3675 2350 50  0000 L CNN
+F 2 "Capacitors_SMD:C_0805" H 3688 2300 50  0001 C CNN
+F 3 "" H 3650 2450 50  0000 C CNN
+	1    3650 2450
+	1    0    0    -1
+$EndComp
+Wire Wire Line
+	2750 2200 2950 2200
+Wire Wire Line
+	2850 2300 2850 2200
+Connection ~ 2850 2200
+Wire Wire Line
+	3550 2200 3750 2200
+Wire Wire Line
+	3650 2300 3650 2200
+Connection ~ 3650 2200
+Wire Wire Line
+	2850 2600 2850 2700
+Wire Wire Line
+	3650 2600 3650 2700
+$Comp
+L GND #PWR029
+U 1 1 58C0D6F3
+P 3650 2700
+F 0 "#PWR029" H 3650 2450 50  0001 C CNN
+F 1 "GND" H 3650 2550 50  0000 C CNN
+F 2 "" H 3650 2700 50  0000 C CNN
+F 3 "" H 3650 2700 50  0000 C CNN
+	1    3650 2700
+	1    0    0    -1
+$EndComp
+$Comp
+L GND #PWR030
+U 1 1 58C0D73E
+P 2850 2700
+F 0 "#PWR030" H 2850 2450 50  0001 C CNN
+F 1 "GND" H 2850 2550 50  0000 C CNN
+F 2 "" H 2850 2700 50  0000 C CNN
+F 3 "" H 2850 2700 50  0000 C CNN
+	1    2850 2700
+	1    0    0    -1
+$EndComp
+Text GLabel 2750 2200 0    60   Input ~ 0
+RX_ANT
+$Comp
+L Q_NMOS_DGS Q2
+U 1 1 58C0DDA2
+P 4500 2200
+F 0 "Q2" H 4800 2250 50  0000 R CNN
+F 1 "Q_NMOS_DGS" H 5150 2150 50  0000 R CNN
+F 2 "TO_SOT_Packages_SMD:SOT-23" H 4700 2300 50  0001 C CNN
+F 3 "" H 4500 2200 50  0000 C CNN
+	1    4500 2200
+	1    0    0    -1
+$EndComp
+$Comp
+L R R11
+U 1 1 58C0DE05
+P 4600 1650
+F 0 "R11" V 4680 1650 50  0000 C CNN
+F 1 "50" V 4600 1650 50  0000 C CNN
+F 2 "Resistors_SMD:R_0603" V 4530 1650 50  0001 C CNN
+F 3 "" H 4600 1650 50  0000 C CNN
+	1    4600 1650
+	1    0    0    -1
+$EndComp
+Wire Wire Line
+	4600 1800 4600 2000
+$Comp
+L C C33
+U 1 1 58C0DE35
+P 4850 1900
+F 0 "C33" H 4875 2000 50  0000 L CNN
+F 1 "10nF" H 4875 1800 50  0000 L CNN
+F 2 "Capacitors_SMD:C_0805" H 4888 1750 50  0001 C CNN
+F 3 "" H 4850 1900 50  0000 C CNN
+	1    4850 1900
+	0    1    1    0
+$EndComp
+Wire Wire Line
+	4700 1900 4600 1900
+Connection ~ 4600 1900
+Wire Wire Line
+	4600 1400 4600 1500
+Wire Wire Line
+	4200 1400 4600 1400
+Wire Wire Line
+	4050 2200 4300 2200
+Wire Wire Line
+	4200 1950 4200 2450
+$Comp
+L R R9
+U 1 1 58C0DEA9
+P 4200 1800
+F 0 "R9" V 4280 1800 50  0000 C CNN
+F 1 "309" V 4200 1800 50  0000 C CNN
+F 2 "Resistors_SMD:R_0603" V 4130 1800 50  0001 C CNN
+F 3 "" H 4200 1800 50  0000 C CNN
+	1    4200 1800
+	1    0    0    -1
+$EndComp
+Wire Wire Line
+	4200 1650 4200 1400
+Connection ~ 4200 2200
+$Comp
+L R R10
+U 1 1 58C0DF03
+P 4200 2600
+F 0 "R10" V 4280 2600 50  0000 C CNN
+F 1 "60.4" V 4200 2600 50  0000 C CNN
+F 2 "Resistors_SMD:R_0603" V 4130 2600 50  0001 C CNN
+F 3 "" H 4200 2600 50  0000 C CNN
+	1    4200 2600
+	1    0    0    -1
+$EndComp
+$Comp
+L R R12
+U 1 1 58C0DF32
+P 4600 2650
+F 0 "R12" V 4680 2650 50  0000 C CNN
+F 1 "4" V 4600 2650 50  0000 C CNN
+F 2 "Resistors_SMD:R_0603" V 4530 2650 50  0001 C CNN
+F 3 "" H 4600 2650 50  0000 C CNN
+	1    4600 2650
+	1    0    0    -1
+$EndComp
+Wire Wire Line
+	4600 2400 4600 2500
+Wire Wire Line
+	4200 2750 4200 2900
+Wire Wire Line
+	4200 2900 4600 2900
+Wire Wire Line
+	4600 2800 4600 3000
+Connection ~ 4600 2900
+$Comp
+L GND #PWR031
+U 1 1 58C0E054
+P 4600 3000
+F 0 "#PWR031" H 4600 2750 50  0001 C CNN
+F 1 "GND" H 4600 2850 50  0000 C CNN
+F 2 "" H 4600 3000 50  0000 C CNN
+F 3 "" H 4600 3000 50  0000 C CNN
+	1    4600 3000
+	1    0    0    -1
+$EndComp
+Wire Wire Line
+	4400 1150 4400 1400
+Connection ~ 4400 1400
+$Comp
+L POT RV2
+U 1 1 58C0E205
+P 3950 1150
+F 0 "RV2" H 3950 1070 50  0000 C CNN
+F 1 "POT" H 3950 1150 50  0000 C CNN
+F 2 "RFBRD:J-FOOT_POT" H 3950 1150 50  0001 C CNN
+F 3 "" H 3950 1150 50  0000 C CNN
+	1    3950 1150
+	0    1    1    0
+$EndComp
+Wire Wire Line
+	4100 1150 4400 1150
+Wire Wire Line
+	3950 1300 3950 1400
+$Comp
+L GND #PWR032
+U 1 1 58C0E29E
+P 3950 1400
+F 0 "#PWR032" H 3950 1150 50  0001 C CNN
+F 1 "GND" H 3950 1250 50  0000 C CNN
+F 2 "" H 3950 1400 50  0000 C CNN
+F 3 "" H 3950 1400 50  0000 C CNN
+	1    3950 1400
+	1    0    0    -1
+$EndComp
+Wire Wire Line
+	3950 1000 3950 900
+Wire Wire Line
+	3950 900  3850 900
+Text GLabel 3850 900  0    60   Input ~ 0
+3V3
+$Comp
+L C C32
+U 1 1 58C0E302
+P 3900 2200
+F 0 "C32" H 3925 2300 50  0000 L CNN
+F 1 "10nF" H 3925 2100 50  0000 L CNN
+F 2 "Capacitors_SMD:C_0805" H 3938 2050 50  0001 C CNN
+F 3 "" H 3900 2200 50  0000 C CNN
+	1    3900 2200
+	0    1    1    0
+$EndComp
+Wire Wire Line
+	5000 1900 5100 1900
+Text GLabel 5100 1900 2    60   Input ~ 0
+RX_IN
 $EndSCHEMATC
