File: hardware/DEMORD/DEMORD.sch (KiCad schematic (older format))
At the start: 4 parts

Commit message: Added further progress to Si4464 Radio Dev Board.
Parts:
- removed X?: 16 MHz, symbol CRYSTAL_SMD
- added C1: 100nF, Capacitors_SMD:C_0805, symbol C
- added C2, C3: 5.6pF, Capacitors_SMD:C_0805, symbol C
- added C4, C5, C6: 10nF, Capacitors_SMD:C_0805, symbol C
- added C7, C8: 20pF, Capacitors_SMD:C_0805, symbol C
- added L1, L3: 43nH, Resistors_SMD:R_0805, symbol L_Small
- added L2: 23nH, Resistors_SMD:R_0805, symbol L_Small
- added L4: 100nH, Resistors_SMD:R_0805, symbol L_Small
- added P1: CONN_01X08, Pin_Headers:Pin_Header_Straight_1x08_Pitch1.27mm, symbol CONN_01X08
- added P2: CONN_01X04, Pin_Headers:Pin_Header_Straight_1x04_Pitch1.27mm, symbol CONN_01X04
- added P3: CONN_01X02, Pin_Headers:Pin_Header_Straight_1x02_Pitch1.27mm, symbol CONN_01X02
- added Y1: 30MHz, Crystals:Crystal_SMD_HC49-SD_HandSoldering, symbol Crystal_Small
- J1: renamed from J?; footprint (none) -> RFBRD:SMA_CONN
- U1: renamed from U?; footprint (none) -> RFBRD:QFN_12_2mmx2mm_0.5PITCH
- U2: renamed from U?; footprint (none) -> Housings_DFN_QFN:QFN-20-1EP_4x4mm_Pitch0.5mm
Connections:
- net labels removed: PWRAMP
- wire segments 22 -> 89
Other:
- moved on the sheet: J1, U1
