File: hardware/pihat/pihat.kicad_pcb (KiCad board)
At the start: 2 copper layers, 85 x 56 mm, 1 part, among them P1 CONN_13X2

Commit message: More updates, improvements, pihat.
Parts:
- added C1: 10uF, Capacitors_SMD:C_0805, F.Cu at (176.5, 182.8)
- added C10: 10uF, Capacitors_SMD:C_0805, F.Cu at (180.5, 194.8)
- added C11: C, Capacitors_SMD:C_0805, F.Cu at (174.5, 144.5)
- added C12: 47uF, Capacitors_SMD:c_elec_5x5.3, F.Cu at (269.8, 114.6)
- added C13: 10uF, Capacitors_SMD:C_0805, F.Cu at (190.2, 198.9)
- added C14: 10uF, Capacitors_SMD:C_0805, F.Cu at (201.1, 196.3)
- added C15: 10uF, Capacitors_SMD:C_0805, F.Cu at (205.4, 196.3)
- added C2: 10uF, Capacitors_SMD:C_0805, F.Cu at (172.1, 199.1)
- added C3: 10uF, Capacitors_SMD:C_0805, F.Cu at (177.7, 199.2)
- added C4: C, Capacitors_SMD:C_0805, F.Cu at (164.0, 152.0)
- added C5: C, Capacitors_SMD:C_0805, F.Cu at (172.0, 153.0)
- added C6: C, Capacitors_SMD:C_0805, F.Cu at (175.5, 152.0)
- added C7: C, Capacitors_SMD:C_0805, F.Cu at (171.5, 144.5)
- added C8: C, Capacitors_SMD:C_0805, F.Cu at (163.5, 143.5)
- added C9: 10uF, Capacitors_SMD:C_0805, F.Cu at (179.4, 189.5)
- added D1: LED, LEDs:LED_0805, F.Cu at (239.1, 130.3)
- added D2: LED, LEDs:LED_0805, F.Cu at (239.0, 120.7)
- added D3: LED, LEDs:LED_0805, F.Cu at (239.0, 125.8)
- added L1: L_Small, Resistors_SMD:R_0805, F.Cu at (168.5, 152.0)
- added L2: L_Small, Resistors_SMD:R_0805, F.Cu at (174.5, 148.5)
- added L3: L_Small, Resistors_SMD:R_0805, F.Cu at (168.0, 143.5)
- added L4: L_Small, Resistors_SMD:R_0805, F.Cu at (178.0, 143.5)
- added L5: 6.8uH, Choke_Axial_ThroughHole:Choke_Horizontal_RM10mm, F.Cu at (253.2, 113.6)
- added L6: 1uH, Choke_Axial_ThroughHole:Choke_Horizontal_RM10mm, F.Cu at (252.6, 121.7)
- added P2: USB_OTG, Connect:USB_Micro-B, F.Cu at (148.0, 178.2)
- added P3: BATT, Pin_Headers:Pin_Header_Straight_1x02, F.Cu at (245.1, 177.0)
- added R1: 1K, Resistors_SMD:R_0805, F.Cu at (190.6, 193.2)
- added R10: R, Resistors_SMD:R_0603, F.Cu at (172.2, 182.8)
- added R11: R, Resistors_SMD:R_0603, F.Cu at (182.1, 199.6)
- added R2: 1K, Resistors_SMD:R_0805, F.Cu at (171.1, 195.2)
- added R3: 1K, Resistors_SMD:R_0805, F.Cu at (186.2, 196.4)
- added R4: 1K, Resistors_SMD:R_0805, F.Cu at (195.1, 195.9)
- added R5: 1K, Resistors_SMD:R_0805, F.Cu at (190.5, 189.2)
- added R6: 150K, Resistors_SMD:R_0603, F.Cu at (175.3, 189.8)
- added R7: R, Resistors_SMD:R_0603, F.Cu at (199.1, 189.9)
- added R8: R, Resistors_SMD:R_0603, F.Cu at (176.7, 195.1)
- added R9: R, Resistors_SMD:R_0603, F.Cu at (200.2, 183.5)
- added RV1: POT, Potentiometers:Potentiometer_Bourns_3296W_3-8Zoll_Inline_ScrewUp, F.Cu at (146.6, 141.3)
- added TH1: 10K, Resistors_SMD:R_0805, F.Cu at (168.5, 183.2)
- added U1: MCP73833, Housings_DFN_QFN:DFN-8-1EP_3x3mm_Pitch0.5mm, F.Cu at (170.9, 190.2)
- added U2: TPS61027, Housings_DFN_QFN:DFN-10-1EP_3x3mm_Pitch0.5mm, F.Cu at (147.2, 170.1)
- added U3: SC189, Housings_DFN_QFN:DFN-6-1EP_2x2mm_Pitch0.5mm, F.Cu at (191.7, 183.2)
- added U4: Si4464, Housings_DFN_QFN:QFN-20-1EP_4x4mm_Pitch0.5mm, F.Cu at (172.1, 137.8)
- added X1: 30MHz, Crystals:Crystal_SMD_5032_4Pads, F.Cu at (164.1, 137.6)
Connections:
- P1 pad 1: +3.3V -> (no net)
- P1 pad 15: (no net) -> VOL
- P1 pad 18: (no net) -> SHDN
- P1 pad 19: (no net) -> SDI
- P1 pad 2: +5V -> 5VU
- P1 pad 21: (no net) -> SDO
- P1 pad 22: (no net) -> nIRQ
- P1 pad 23: (no net) -> SCLK
- P1 pad 24: (no net) -> nSEL
Routing:
- net VOL: track 0.00 -> 26.6 mm
- net nSEL: track 0.00 -> 24.5 mm, vias 0 -> 1
- net nIRQ: track 0.00 -> 21.4 mm
- net 5VU: track 0.00 -> 15.7 mm
- net SHDN: track 0.00 -> 13.1 mm
- net Net-(U4-Pad17): track 0.00 -> 9.02 mm
- net SDI: track 0.00 -> 7.69 mm
- net Net-(C8-Pad2): track 0.00 -> 7.68 mm
- net SCLK: track 0.00 -> 6.04 mm
- net SDO: track 0.00 -> 5.93 mm
- net Net-(C6-Pad1): track 0.00 -> 5.10 mm
- net Net-(C4-Pad1): track 0.00 -> 5.10 mm
- net Net-(C11-Pad1): track 0.00 -> 4.78 mm
- net Net-(U4-Pad16): track 0.00 -> 4.15 mm
- net Net-(C7-Pad1): track 0.00 -> 3.84 mm
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