File: hardware/RF BW Filter/RF BW Filter/RF BW Filter.kicad_pcb (KiCad board)
At the start: 2 copper layers, 52 x 23.5 mm, 7 parts, among them U1 SMA_Edge_Mount, U2 SMA_Edge_Mount

Commit message: tweaks for better pcb
Parts:
- moved C1 11.4 mm to (135.2, 107.0)
- moved C2 11.0 mm to (147.2, 107.0)
- moved C3 10.8 mm to (160.0, 107.0)
Routing:
- net GND: track 203.7 -> 104.4 mm, vias 50 -> 3
- net (no net): track 0.00 -> 79.6 mm, vias 0 -> 28
- net Net-(C3-Pad1): track 38.6 -> 14.8 mm
- net Net-(C2-Pad1): track 32.7 -> 11.1 mm
- net Net-(C1-Pad1): track 37.3 -> 16.3 mm
Other:
- board size 52 x 23.5 mm -> 52 x 12 mm
