File: hardware/PiHat_Final/HAT.sch (KiCad schematic (older format))
At the start: 41 parts

Commit message: Added more to the Schematic.
Parts:
- removed C? (x6): C, Capacitors_SMD:C_0805, symbol C
- removed C? (x2): 10nF, Capacitors_SMD:C_0805, symbol C
- removed L? (x4): L_Small, Resistors_SMD:R_0805, symbol L_Small
- removed R? (x5): R, Resistors_SMD:R_0603, symbol R
- removed RV?: POT, Potentiometers:Potentiometer_Bourns_3296W_3-8Zoll_Inline_ScrewUp, symbol POT
- removed U?: Si4464, Housings_DFN_QFN:QFN-20-1EP_4x4mm_Pitch0.5mm, symbol Si4464
- removed X?: 30MHz, Crystals:Crystal_SMD_5032_4Pads, symbol CRYSTAL_SMD
- added SW1: PWR_VOL, symbol ROTARY_ENCODER_SWITCH
- gave numbers to parts that had none: 21
Connections:
- net +5V: now also SW1.1 (A)
- net GND: now also SW1.3 (B)
- net VBAT: now also SW1.5; no longer C2.1, P2.2 (P2), U2.10 (VBAT), U2.9 (VBAT)
- net VOL: now also SW1.2 (C)
- new net VBP_SW: C2.1, P2.2 (P2), SW1.4, U2.10 (VBAT), U2.9 (VBAT)
- no-connect marks 8 -> 6

Commit message: PCB Layout Changes
minor changes, will continue layout
Parts:
- D1, D2, D3: symbol LED -> LED-RESCUE-RPi_Hat
- P1: symbol USB_OTG -> USB_OTG-RESCUE-RPi_Hat
- SW1: footprint (none) -> rotary_potentiometer:rotary_potentiometer
Changed lines of the file:
@@
 EESchema Schematic File Version 2
+LIBS:RPi_Hat-rescue
 LIBS:power
 LIBS:device
@@
 $EndDescr
 $Comp
-L USB_OTG P1
+L USB_OTG-RESCUE-RPi_Hat P1
 U 1 1 58E977AB
 P 850 3900
@@
 $EndComp
 $Comp
-L LED D2
+L LED-RESCUE-RPi_Hat D2
 U 1 1 58E977B5
 P 2600 3300
+AR Path="/58E977B5" Ref="D2"  Part="1"
+AR Path="/58E9654B/58E977B5" Ref="D2"  Part="1"
 F 0 "D2" H 2600 3400 50  0000 C CNN
 F 1 "LED" H 2600 3200 50  0000 C CNN
@@
 $EndComp
 $Comp
-L LED D1
+L LED-RESCUE-RPi_Hat D1
 U 1 1 58E977B7
 P 2300 3300
+AR Path="/58E977B7" Ref="D1"  Part="1"
+AR Path="/58E9654B/58E977B7" Ref="D1"  Part="1"
 F 0 "D1" H 2300 3400 50  0000 C CNN
 F 1 "LED" H 2300 3200 50  0000 C CNN
@@
 	4600 3100 4600 3000
 $Comp
-L LED D3
+L LED-RESCUE-RPi_Hat D3
 U 1 1 58E977BC
 P 4400 3000
+AR Path="/58E977BC" Ref="D3"  Part="1"
+AR Path="/58E9654B/58E977BC" Ref="D3"  Part="1"
 F 0 "D3" H 4400 3100 50  0000 C CNN
 F 1 "LED" H 4400 2900 50  0000 C CNN
@@
 F 0 "SW1" H 1150 6660 50  0000 C CNN
 F 1 "PWR_VOL" H 1150 6140 50  0000 C CNN
-F 2 "" H 1050 6560 50  0001 C CNN
+F 2 "rotary_potentiometer:rotary_potentiometer" H 1050 6560 50  0001 C CNN
 F 3 "" H 1150 6660 50  0001 C CNN
 	1    1150 6400
